File: Hardware/SparkFun_QwiicBus_Endpoint.sch (EAGLE design)
At the start: 39 parts, among them J1 QWIIC, J2 QWIIC, J3 RJ45, U1 PCA9615

Commit message: post FarmHand Review
Parts:
- removed J7: (no value), SparkFun-Connectors:CONN_021X02_NO_SILK
- added 0-1: JUMPER-SMT_2_NC_TRACE_SILK, SparkFun-Jumpers:JUMPER-SMT_2_NC_TRACE_SILK
- added J4, J6: (no value), SparkFun-Connectors:CONN_041X04_NO_SILK
- LOGO5: value SFE_LOGO_NAME.1_INCH -> SFE_LOGO_FLAME.1_INCH; device SparkFun-Aesthetics:SFE_LOGO_NAME.1_INCH -> SparkFun-Aesthetics:SFE_LOGO_FLAME.1_INCH
- renumbered VDDA to VCC1
Connections:
- removed net 3.3V: C1.1, C2.1, C3.1, C4.1, D11.A, I2C.2, J1.2, J2.2, J8.2, R1.2, R4.2, U1.VDDA, U1.VDDB, VCC1.1
- new net VCC: 0-1.2, C1.1, C3.1, D11.A, I2C.2, J1.2, J2.2, J8.2, U1.VDDA
- new net VCC_1: 0-1.1, C2.1, C4.1, J4.2, J6.2, R1.2, R4.2, U1.VDDB, VCC1.1
- net GND: now also J4.1, J6.1
- net GRN_N: now also J4.3, J6.3; no longer J7.1
- net GRN_P: now also J4.4, J6.4; no longer J7.2
Other:
- note added: "Cut 0-1 Jumper to provide separate voltage to VCC1"
- note added: "Cut traces on VCC1 and GND jumpers to disconnect VCC1 and GND from cable."
- note added: "VCC: I2C-bus side power supply (2.3V-5.5V) VCC1: Differential side power supply (3.0V-5.5V)"
- note removed: "Cut traces on VDDA and GND jumpers to disconnect VDDA and GND from cable."
- moved on the sheet: J5, J8

Commit message: post checklist changes
Other:
- note added: "Cut 0-1 Jumper to provide separate voltage to VCC1 and VCC (VCC0)"
- note added: "Depending on load and distance requirements, there are several different ways to power the Midpoint/Endpoint combo. --- The default option powers the entire system using 3.3V, in this configuration, the BP jumper is closed and both sides of the PSEL jumper are open. --- To power the VCC_1 rail with 5V (The PCA9615 operates better at this voltage), the BP jumper must be opened. Then close the "1" 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"
- note removed: "Cut 0-1 Jumper to provide separate voltage to VCC1"
Changed lines of the file:
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@@
 jumper to disable
 the PWR LED</text>
-<text x="5.08" y="177.8" size="1.778" layer="94">VIN: 3.0-5.5V</text>
+<text x="5.08" y="177.8" size="1.778" layer="94" font="vector">VIN: 3.0-5.5V</text>
 <text x="5.08" y="101.6" size="1.778" layer="94" font="vector">VCC: I2C-bus side power supply (2.3V-5.5V)
 VCC1: Differential side power supply (3.0V-5.5V)</text>
 <text x="15.24" y="167.64" size="1.778" layer="94" font="vector">Cut 0-1 Jumper to provide
-separate voltage to VCC1</text>
+separate voltage to VCC1 and VCC
+(VCC0)</text>
+<text x="91.44" y="93.98" size="1.27" layer="97" font="vector">Depending on load and distance requirements, there are several different ways to power the Midpoint/Endpoint combo.
+---
+The default option powers the entire system using 3.3V, in this configuration, the BP jumper is closed and both sides of the PSEL jumper are open.
+---
+To power the VCC_1 rail with 5V (The PCA9615 operates better at this voltage), the BP jumper must be opened. Then close the "1" side of
+the PSEL jumper. Also ensure that 5V is connected on the VCC_1 pin on the Qwiic Endpoint
+---
+If many devices need to be powered, it is possible to send up to 36V over the green pair. To do this, connect 36V and ground to the Qwiic
+Endpoint. Also make sure that the BP jumper is cut/open. Make sure the 1 side of the PSEL jumper is open and close the 2 side of the
+PSEL jumper</text>
 </plain>
 <instances>
