File: Hardware/SparkFun_QwiicBus_Endpoint.brd (EAGLE design)
At the start: 44.5 x 25.4 mm, 61 parts, among them J1 QWIIC, J2 QWIIC, J3 RJ45, U1 PCA9615

Commit message: post FarmHand Review
Parts:
- removed J7: (no value), SparkFun-Connectors:1X02_NO_SILK
- added 0-1: JUMPER-SMT_2_NC_TRACE_SILK, SparkFun-Jumpers:SMT-JUMPER_2_NC_TRACE_SILK
- added J4, J6: (no value), SparkFun-Connectors:1X04_NO_SILK
- added U$14, U$2, U$29, U$30: (no value), output:GRN0
- added U$18, U$22, U$24: (no value), output:#GRNW#0
- added U$20, U$31, U$32: (no value), output:#VCC1#0
- added U$33, U$34: (no value), output:#GND#0
- added U$35: (no value), output:ENDPOINT0
- LOGO5: value SFE_LOGO_NAME.1_INCH -> SFE_LOGO_FLAME.1_INCH; device SparkFun-Aesthetics:SFE_LOGO_NAME_.1 -> SparkFun-Aesthetics:SFE_LOGO_FLAME_.1
- U$13: device output:#HV##1 -> output:#GND#0
- U$21: device output:#GRN#0 -> output:#VCC1#0
- U$25: device output:ENDPOINT0 -> output:0#10
- U$3: device output:#HV##0 -> output:#GND#0
- moved U$25 19.6 mm to (17.3, 17.0)
- moved LOGO5 17.2 mm to (20.4, 20.4)
- moved U$19 6.89 mm to (36.1, 1.27), turned to 0 degrees
- moved U$21 3.82 mm to (30.5, 1.78), flipped to the bottom
- moved U$13 1.27 mm to (27.9, 1.78)
- moved U$3 1.27 mm to (27.9, 1.78), flipped to the top
- renumbered VDDA to VCC1
Connections:
- removed net 3.3V: C1.1, C2.1, C3.1, C4.1, D11.A, I2C.2, J1.2, J2.2, J8.2, R1.2, R4.2, U1.1, U1.10, VCC1.1
- new net VCC: 0-1.2, C1.1, C3.1, D11.A, I2C.2, J1.2, J2.2, J8.2, U1.1
- new net VCC_1: 0-1.1, C2.1, C4.1, J4.2, J6.2, R1.2, R4.2, U1.10, VCC1.1
- net GND: now also J4.1, J6.1
- net GRN_N: now also J4.3, J6.3; no longer J7.1
- net GRN_P: now also J4.4, J6.4; no longer J7.2
Routing:
- net 3.3V: track 79.9 -> 0.00 mm, vias 4 -> 0
- net VCC_1: track 0.00 -> 53.8 mm, vias 0 -> 2
- net VCC: track 0.00 -> 47.7 mm, vias 0 -> 2
- net GRN_P: track 14.5 -> 25.5 mm
- net GRN_N: track 17.5 -> 27.6 mm

Commit message: updating silk as per double check
Parts:
- U$14: device output:GRN0 -> output:#GND2#0
- U$18: device output:#GRNW#0 -> output:#GND2#0
- U$24: device output:#GRNW#0 -> output:#VCC2#0
- U$30: device output:GRN0 -> output:#VCC2#0
- moved U$24 23.3 mm to (35.6, 1.78), turned to 90 degrees
- moved U$14 20.7 mm to (33.0, 23.6), turned to 270 degrees
- moved U$18 7.64 mm to (33.0, 1.78), turned to 90 degrees
- moved U$30 1.57 mm to (35.6, 23.6), turned to 270 degrees
Changed lines of the file:
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@@
 </element>
 <element name="U$2" library="output" package="GRN0" value="" x="30.861" y="3.048" smashed="yes"/>
-<element name="U$14" library="output" package="GRN0" value="" x="35.179" y="3.048" smashed="yes" rot="MR0"/>
-<element name="U$18" library="output" package="#GRNW#0" value="" x="40.64" y="1.27" smashed="yes" rot="MR0"/>
 <element name="U$3" library="output" package="#GND#0" value="" x="27.94" y="1.778" smashed="yes" rot="R90"/>
 <element name="U$13" library="output" package="#GND#0" value="" x="27.94" y="1.778" smashed="yes" rot="MR90"/>
@@
 </element>
 <element name="U$22" library="output" package="#GRNW#0" value="" x="36.322" y="24.13" smashed="yes"/>
-<element name="U$24" library="output" package="#GRNW#0" value="" x="42.164" y="24.13" smashed="yes" rot="MR0"/>
 <element name="U$29" library="output" package="GRN0" value="" x="30.861" y="22.098" smashed="yes"/>
-<element name="U$30" library="output" package="GRN0" value="" x="35.179" y="22.098" smashed="yes" rot="MR0"/>
 <element name="U$31" library="output" package="#VCC1#0" value="" x="30.48" y="23.622" smashed="yes" rot="MR270"/>
 <element name="U$32" library="output" package="#VCC1#0" value="" x="30.48" y="23.622" smashed="yes" rot="R270"/>
@@
 <element name="LOGO5" library="SparkFun-Aesthetics" package="SFE_LOGO_FLAME_.1" value="SFE_LOGO_FLAME.1_INCH" x="20.447" y="20.447" smashed="yes"/>
 <element name="U$25" library="output" package="0#10" value="" x="17.272" y="17.018" smashed="yes"/>
+<element name="U$14" library="output" package="#GND2#0" value="" x="33.02" y="23.622" smashed="yes" rot="MR270"/>
+<element name="U$18" library="output" package="#GND2#0" value="" x="33.02" y="1.778" smashed="yes" rot="MR90"/>
+<element name="U$24" library="output" package="#VCC2#0" value="" x="35.56" y="1.778" smashed="yes" rot="MR90"/>
+<element name="U$30" library="output" package="#VCC2#0" value="" x="35.56" y="23.622" smashed="yes" rot="MR270"/>
 </elements>
 <signals>
